File: pcb_d6/pcb_d6.kicad_pcb (KiCad board)
At the start: 2 copper layers, 22 parts, among them J1 Conn_01x06, SW1 SW_Push, U1 ATtiny13A-S

Commit message: PCB redesigned
Parts:
- moved R1 21.1 mm to (92.5, 134.4)
Connections:
- J1 pad 5: /PB5 -> /LED1
- R1 pad 1: /PB5 -> /LIGHT
- R2 pad 2: /PB5 -> /LIGHT
- U1 pad 1: /PB5 -> /LED1
- U1 pad 2: /LED1 -> /LIGHT
Routing:
- net /LED1: track 116.7 -> 147.7 mm
- net /PB5: track 28.9 -> 0.00 mm
- net /LIGHT: track 0.00 -> 26.1 mm
- net Net-(U1-PB4): track 16.4 -> 17.5 mm
Other:
- board text added: "hát ezt karczolja a szivats"
