File: pcb_d6/pcb_d6.kicad_sch (KiCad schematic)
At the start: 22 parts, among them J1 Conn_01x06, SW1 SW_Push, U1 ATtiny13A-S

Commit message: PCB done
Parts:
- removed D1: D_Photo_Filled, symbol Device:D_Photo_Filled
- added R10: R, Resistor_SMD:R_1206_3216Metric, symbol Device:R
- BT1: footprint (none) -> Battery:BatteryHolder_Keystone_103_1x20mm
- D2, D3, D4, D5, D6, D7, D8: footprint (none) -> FootPrints:LED_4
- J1: footprint (none) -> Connector_PinHeader_2.54mm:PinHeader_1x06_P2.54mm_Vertical
- R2: footprint (none) -> FootPrints:R_PHOTO_2
- SW1: footprint (none) -> FootPrints:BUTTON_4
Connections:
- net LED1: now also D3.2 (A), D8.2 (A), U1.2 (PB3); no longer D5.2 (A), J1.2 (Pin_2), U1.5 (PB0)
- net LED3: now also R10.1, R10.2
- net LED4: now also D5.2 (A), J1.2 (Pin_2), U1.5 (PB0); no longer D3.2 (A), D8.2 (A), U1.2 (PB3)
- net PB5: now also R2.2
- net VCC: now also BT1.1 (+), C1.1

Commit message: PCB redesigned
Connections:
- net LED1: now also J1.5 (Pin_5), U1.1 (~{RESET}/PB5); no longer U1.2 (PB3)
- net PB5 renamed LIGHT
- net LIGHT: now also U1.2 (PB3); no longer J1.5 (Pin_5), U1.1 (~{RESET}/PB5)
Changed lines of the file:
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@@
     (effects (font (size 1.27 1.27)) (justify left bottom))
   )
-  (label "PB5" (at 46.99 96.52 0) (fields_autoplaced)
+  (label "LED1" (at 46.99 96.52 0) (fields_autoplaced)
     (effects (font (size 1.27 1.27)) (justify left bottom))
   )
-  (label "LED1" (at 163.83 101.6 0) (fields_autoplaced)
+  (label "LIGHT" (at 163.83 101.6 0) (fields_autoplaced)
     (effects (font (size 1.27 1.27)) (justify left bottom))
   )
@@
     (effects (font (size 1.27 1.27)) (justify left bottom))
   )
-  (label "PB5" (at 91.44 64.77 0) (fields_autoplaced)
+  (label "LIGHT" (at 91.44 64.77 0) (fields_autoplaced)
     (effects (font (size 1.27 1.27)) (justify left bottom))
   )
@@
     (effects (font (size 1.27 1.27)) (justify left bottom))
   )
-  (label "PB5" (at 163.83 106.68 0) (fields_autoplaced)
+  (label "LED1" (at 163.83 106.68 0) (fields_autoplaced)
     (effects (font (size 1.27 1.27)) (justify left bottom))
   )
